File: schematics/ZComputer-Main/ZComputer-Main.kicad_sch (KiCad schematic)
At the start: 3 parts, among them J1 Board to board connector, U1 74HC137

Commit message: Main board: Add PCB layout
Signed-off-by: Maxime Chretien <mchretien@linuxmail.org>
Parts:
- C1: footprint (none) -> Capacitor_THT:C_Disc_D4.3mm_W1.9mm_P5.00mm
- J1: footprint (none) -> Connector_PinSocket_2.54mm:PinSocket_2x34_P2.54mm_Horizontal
- U1: footprint (none) -> Package_DIP:DIP-16_W7.62mm_Socket_LongPads
Changed lines of the file:
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@@
 	(label "D4"
 		(at 33.02 66.04 0)
+		(fields_autoplaced yes)
 		(effects
 			(font
@@
 	(label "D7"
 		(at 33.02 73.66 0)
+		(fields_autoplaced yes)
 		(effects
 			(font
@@
 	(label "D2"
 		(at 33.02 60.96 0)
+		(fields_autoplaced yes)
 		(effects
 			(font
@@
 	(label "D3"
 		(at 33.02 63.5 0)
+		(fields_autoplaced yes)
 		(effects
 			(font
@@
 	(label "D1"
 		(at 33.02 58.42 0)
+		(fields_autoplaced yes)
 		(effects
 			(font
@@
 	(label "D6"
 		(at 33.02 71.12 0)
+		(fields_autoplaced yes)
 		(effects
 			(font
@@
 	(label "D5"
 		(at 33.02 68.58 0)
+		(fields_autoplaced yes)
 		(effects
 			(font
@@
 	(label "D0"
 		(at 33.02 55.88 0)
+		(fields_autoplaced yes)
 		(effects
 			(font
@@
 			)
 		)
-		(property "Footprint" ""
+		(property "Footprint" "Connector_PinSocket_2.54mm:PinSocket_2x34_P2.54mm_Horizontal"
 			(at 45.72 91.44 0)
 			(effects
@@
 			)
 		)
-		(property "Footprint" ""
+		(property "Footprint" "Capacitor_THT:C_Disc_D4.3mm_W1.9mm_P5.00mm"
 			(at 243.84 75.8952 0)
 			(effects
@@
 			)
 		)
-		(property "Footprint" ""
+		(property "Footprint" "Package_DIP:DIP-16_W7.62mm_Socket_LongPads"
 			(at 238.76 93.98 0)
 			(effects
